File: core/power/crowbar/crowbar.kicad_pcb (KiCad board)
At the start: 2 copper layers, 0 parts

Commit message: Finished crowbar and generated mfg files
Parts:
- added D1: LM431, TO_SOT_Packages_SMD:SOT-23_Handsoldering, F.Cu at (109.3, 74.6)
- added D2: RED, LEDs:LED-5MM, F.Cu at (109.4, 65.3)
- added F1: 3A, C-BISCUIT:3549-BLADE-CLIP, B.Cu at (109.1, 63.3)
- added P1: CONN_01X01, Wire_Pads:SolderWirePad_single_SMD_5x10mm, F.Cu at (109.2, 52.8)
- added P2: CONN_01X01, Wire_Pads:SolderWirePad_single_SMD_5x10mm, F.Cu at (109.2, 83.0)
- added P3: CONN_01X01, Wire_Pads:SolderWirePad_single_SMD_5x10mm, B.Cu at (109.2, 83.0)
- added P4: CONN_01X01, Wire_Pads:SolderWirePad_single_SMD_5x10mm, B.Cu at (109.2, 52.8)
- added R1: 3.48K, Resistors_SMD:R_0805_HandSoldering, F.Cu at (112.2, 74.6)
- added R2: 2.49K, Resistors_SMD:R_0805_HandSoldering, F.Cu at (109.3, 78.4)
- added R3: 200, Resistors_SMD:R_0805_HandSoldering, F.Cu at (114.0, 63.2)
- added R4: 220, Resistors_SMD:R_0805_HandSoldering, F.Cu at (106.5, 74.6)
- added U1: BT137S, TO_SOT_Packages_SMD:TO-252-2Lead, B.Cu at (113.2, 75.4)
Routing:
- net /DEVICE: track 0.00 -> 49.0 mm
- net (no net): track 0.00 -> 17.8 mm
- net /SUPPLY: track 0.00 -> 17.2 mm
- net Net-(D1-Pad1): track 0.00 -> 11.9 mm, vias 0 -> 1
- net GND: track 0.00 -> 11.5 mm, vias 0 -> 2
- net Net-(D2-Pad2): track 0.00 -> 4.99 mm
- net Net-(D1-Pad2): track 0.00 -> 4.18 mm
- added copper zone on B.Cu, net GND
Other:
- board outline added: 13 x 37.2 mm
- board text added: "C-BISCUIT 5V Crowbar"
- board text added: "DEV"
- board text added: "GND"
- board text added: "SUPPLY"

Commit message: Finished crowbar article and mfg files
Parts:
- added REF**: Symbol_OSHW-Logo_SilkScreen, C-BISCUIT:Symbol_OSHW-Logo_SilkScreen_NoLetters, B.Cu at (105.8, 63.2)
Changed lines of the file:
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@@
-(kicad_pcb (version 4) (host pcbnew 0.201602231446+6579~42~ubuntu15.04.1-product)
+(kicad_pcb (version 4) (host pcbnew 0.201602271447+6593~42~ubuntu15.04.1-product)
   (general
     (links 18)
     (no_connects 0)
-    (area 100.474999 47.691666 118.925002 88.108333)
+    (area 100.28588 47.691666 118.925002 88.108333)
     (thickness 1.6)
     (drawings 13)
     (tracks 44)
     (zones 0)
-    (modules 12)
+    (modules 13)
     (nets 7)
   )
@@
     (descr http://www.keyelco.com/product-pdf.cfm?p=303)
     (tags fuse)
-    (fp_text reference F1 (at 0.265 -3.32 180) (layer B.SilkS)
+    (fp_text reference F1 (at -0.135 6.88 180) (layer B.SilkS)
       (effects (font (size 1 1) (thickness 0.15)) (justify mirror))
     )
@@
       (net 6 /SUPPLY))
   )
+  (module C-BISCUIT:Symbol_OSHW-Logo_SilkScreen_NoLetters (layer B.Cu)
+    (at 105.8 63.2 270)
+    (descr "Symbol, OSHW-Logo, Silk Screen,")
+    (tags "Symbol, OSHW-Logo, Silk Screen,")
+    (fp_text reference REF** (at 0.09906 4.38912 270) (layer B.SilkS) hide
+      (effects (font (size 1 1) (thickness 0.15)) (justify mirror))
+    )
+    (fp_text value Symbol_OSHW-Logo_SilkScreen (at 0.30988 -6.56082 270) (layer B.Fab)
+      (effects (font (size 1 1) (thickness 0.15)) (justify mirror))
+    )
+    (fp_line (start -1.78054 -0.92964) (end -2.03962 -1.49098) (layer B.SilkS) (width 0.15))
+    (fp_line (start -2.03962 -1.49098) (end -1.50114 -2.00914) (layer B.SilkS) (width 0.15))
+    (fp_line (start -1.50114 -2.00914) (end -0.98044 -1.7399) (layer B.SilkS) (width 0.15))
+    (fp_line (start -0.98044 -1.7399) (end -0.70104 -1.89992) (layer B.SilkS) (width 0.15))
+    (fp_line (start 0.73914 -1.8796) (end 1.06934 -1.6891) (layer B.SilkS) (width 0.15))
+    (fp_line (start 1.06934 -1.6891) (end 1.50876 -2.0193) (layer B.SilkS) (width 0.15))
+    (fp_line (start 1.50876 -2.0193) (end 1.9812 -1.52908) (layer B.SilkS) (width 0.15))
+    (fp_line (start 1.9812 -1.52908) (end 1.69926 -1.04902) (layer B.SilkS) (width 0.15))
+    (fp_line (start 1.69926 -1.04902) (end 1.88976 -0.57912) (layer B.SilkS) (width 0.15))
+    (fp_line (start 1.88976 -0.57912) (end 2.49936 -0.39116) (layer B.SilkS) (width 0.15))
+    (fp_line (start 2.49936 -0.39116) (end 2.49936 0.28956) (layer B.SilkS) (width 0.15))
+    (fp_line (start 2.49936 0.28956) (end 1.94056 0.42926) (layer B.SilkS) (width 0.15))
+    (fp_line (start 1.94056 0.42926) (end 1.7399 1.00076) (layer B.SilkS) (width 0.15))
+    (fp_line (start 1.7399 1.00076) (end 2.00914 1.47066) (layer B.SilkS) (width 0.15))
+    (fp_line (start 2.00914 1.47066) (end 1.53924 1.9812) (layer B.SilkS) (width 0.15))
+    (fp_line (start 1.53924 1.9812) (end 1.02108 1.71958) (layer B.SilkS) (width 0.15))
+    (fp_line (start 1.02108 1.71958) (end 0.55118 1.92024) (layer B.SilkS) (width 0.15))
+    (fp_line (start 0.55118 1.92024) (end 0.381 2.46126) (layer B.SilkS) (width 0.15))
+    (fp_line (start 0.381 2.46126) (end -0.30988 2.47904) (layer B.SilkS) (width 0.15))
+    (fp_line (start -0.30988 2.47904) (end -0.5207 1.9304) (layer B.SilkS) (width 0.15))
+    (fp_line (start -0.5207 1.9304) (end -0.9398 1.76022) (layer B.SilkS) (width 0.15))
+    (fp_line (start -0.9398 1.76022) (end -1.49098 2.02946) (layer B.SilkS) (width 0.15))
+    (fp_line (start -1.49098 2.02946) (end -2.00914 1.50114) (layer B.SilkS) (width 0.15))
+    (fp_line (start -2.00914 1.50114) (end -1.76022 0.96012) (layer B.SilkS) (width 0.15))
+    (fp_line (start -1.76022 0.96012) (end -1.9304 0.48006) (layer B.SilkS) (width 0.15))
+    (fp_line (start -1.9304 0.48006) (end -2.47904 0.381) (layer B.SilkS) (width 0.15))
+    (fp_line (start -2.47904 0.381) (end -2.4892 -0.32004) (layer B.SilkS) (width 0.15))
+    (fp_line (start -2.4892 -0.32004) (end -1.9304 -0.5207) (layer B.SilkS) (width 0.15))
+    (fp_line (start -1.9304 -0.5207) (end -1.7907 -0.91948) (layer B.SilkS) (width 0.15))
+    (fp_line (start 0.35052 -0.89916) (end 0.65024 -0.7493) (layer B.SilkS) (width 0.15))
+    (fp_line (start 0.65024 -0.7493) (end 0.8509 -0.55118) (layer B.SilkS) (width 0.15))
+    (fp_line (start 0.8509 -0.55118) (end 1.00076 -0.14986) (layer B.SilkS) (width 0.15))
+    (fp_line (start 1.00076 -0.14986) (end 1.00076 0.24892) (layer B.SilkS) (width 0.15))
+    (fp_line (start 1.00076 0.24892) (end 0.8509 0.59944) (layer B.SilkS) (width 0.15))
+    (fp_line (start 0.8509 0.59944) (end 0.39878 0.94996) (layer B.SilkS) (width 0.15))
+    (fp_line (start 0.39878 0.94996) (end -0.0508 1.00076) (layer B.SilkS) (width 0.15))
+    (fp_line (start -0.0508 1.00076) (end -0.44958 0.89916) (layer B.SilkS) (width 0.15))
+    (fp_line (start -0.44958 0.89916) (end -0.8509 0.55118) (layer B.SilkS) (width 0.15))
+    (fp_line (start -0.8509 0.55118) (end -1.00076 0.09906) (layer B.SilkS) (width 0.15))
+    (fp_line (start -1.00076 0.09906) (end -0.94996 -0.39878) (layer B.SilkS) (width 0.15))
+    (fp_line (start -0.94996 -0.39878) (end -0.70104 -0.70104) (layer B.SilkS) (width 0.15))
+    (fp_line (start -0.70104 -0.70104) (end -0.35052 -0.89916) (layer B.SilkS) (width 0.15))
+    (fp_line (start -0.35052 -0.89916) (end -0.70104 -1.89992) (layer B.SilkS) (width 0.15))
+    (fp_line (start 0.35052 -0.89916) (end 0.7493 -1.89992) (layer B.SilkS) (width 0.15))
+  )
   (gr_text GND (at 113.4 79.8) (layer B.SilkS)
     (effects (font (size 0.9 0.9) (thickness 0.18)) (justify mirror))
   )
-  (gr_text GND (at 109.4 57.2) (layer B.SilkS)
+  (gr_text GND (at 109.2 57.2) (layer B.SilkS)
     (effects (font (size 1 1) (thickness 0.2)) (justify mirror))
   )
