File: core/power/crowbar/crowbar.sch (KiCad schematic (older format))
At the start: 14 parts

Commit message: Finished crowbar and generated mfg files
Parts:
- removed MH1, MH2, MH3, MH4: MOUNTING_HOLE, C-BISCUIT:Mounting_Hole_M3x0.5L_~Plate~_~Pad~, symbol CONN_01X01
- added D2: RED, LEDs:LED-5MM, symbol LED
- added R3: 200, Resistors_SMD:R_0805_HandSoldering, symbol R
- F1: footprint Fuse_Holders_and_Fuses:Fuse_SMD1206_HandSoldering -> C-BISCUIT:3549-BLADE-CLIP
- P1, P2, P3, P4: renamed from P?; footprint (none) -> Wire_Pads:SolderWirePad_single_SMD_5x10mm
- gave numbers to parts that had none: 1
- renumbered D2 to D1, R6 to R1, R7 to R2, R10 to R4
Connections:
- net GND: now also D2.1 (K)
- net DEV_IN renamed DEVICE
- net DEVICE: now also R3.1
- net REG_OUT renamed SUPPLY
- new net: D2.2 (A), R3.2
- no-connect marks 4 -> 0
Other:
- note removed: "36-3550-ND Blade Fuse Clips (ATO)"
- moved on the sheet: P1, P2, P3, P4

Commit message: Finished crowbar article and mfg files
Parts:
- R4: value 220 -> 200
Changed lines of the file:
@@
 P 5200 5250
 F 0 "R4" H 5270 5296 50  0000 L CNN
-F 1 "220" H 5270 5204 50  0000 L CNN
+F 1 "200" H 5270 5204 50  0000 L CNN
 F 2 "Resistors_SMD:R_0805_HandSoldering" V 5130 5250 50  0001 C CNN
 F 3 "" H 5200 5250 50  0000 C CNN
@@
 $EndComp
 $Comp
-L GND #PWR3
+L GND #PWR01
 U 1 1 56A29EAD
 P 4950 6150
-F 0 "#PWR3" H 4950 5900 50  0001 C CNN
+F 0 "#PWR01" H 4950 5900 50  0001 C CNN
 F 1 "GND" H 4958 5976 50  0000 C CNN
 F 2 "" H 4950 6150 50  0000 C CNN
@@
 DEVICE
 Wire Wire Line
-	4700 5050 4850 5050
-Wire Wire Line
-	4850 5050 5000 5050
-Wire Wire Line
-	5000 5050 5200 5050
-Wire Wire Line
-	5200 5050 5800 5050
-Wire Wire Line
-	5800 5050 6150 5050
+	4700 5050 6150 5050
 Wire Wire Line
 	4850 5050 4850 5150
@@
 Connection ~ 4850 5700
 Wire Wire Line
-	4850 5450 4850 5700
-Wire Wire Line
-	4850 5700 4850 5750
+	4850 5450 4850 5750
 Wire Wire Line
 	4850 6050 4850 6100
@@
 	5800 6100 5800 5800
 Wire Wire Line
-	4850 6100 4950 6100
-Wire Wire Line
-	4950 6100 5200 6100
-Wire Wire Line
-	5200 6100 5800 6100
+	4850 6100 5800 6100
 Connection ~ 5800 5050
 Wire Wire Line
@@
 	5200 5050 5200 5100
 Wire Wire Line
-	5200 5400 5200 5450
-Wire Wire Line
-	5200 5450 5200 5500
+	5200 5400 5200 5500
 $Comp
 L BT137S U1
@@
 $EndComp
 $Comp
-L GND #PWR1
+L GND #PWR02
 U 1 1 56CE7583
 P 7150 5800
-F 0 "#PWR1" H 7150 5550 50  0001 C CNN
+F 0 "#PWR02" H 7150 5550 50  0001 C CNN
 F 1 "GND" H 7158 5626 50  0000 C CNN
 F 2 "" H 7150 5800 50  0000 C CNN
@@
 $EndComp
 $Comp
-L GND #PWR2
+L GND #PWR03
 U 1 1 56CE7830
 P 7150 6150
-F 0 "#PWR2" H 7150 5900 50  0001 C CNN
+F 0 "#PWR03" H 7150 5900 50  0001 C CNN
 F 1 "GND" H 7158 5976 50  0000 C CNN
 F 2 "" H 7150 6150 50  0000 C CNN
@@
 $EndComp
 $Comp
-L GND #PWR4
+L GND #PWR04
 U 1 1 56D0AB0A
 P 5850 4700
-F 0 "#PWR4" H 5850 4450 50  0001 C CNN
+F 0 "#PWR04" H 5850 4450 50  0001 C CNN
 F 1 "GND" H 5858 4526 50  0000 C CNN
 F 2 "" H 5850 4700 50  0000 C CNN
